File: Alimentação.kicad_sch (KiCad schematic)
At the start: 13 parts, among them U1 Lm2596 DC-DC Buck, U2 XL4015

Commit message: Mudanças nos footprints
Parts:
- U1: footprint Footprints Personalizados:Lm2596 -> Footprints Personalizados:Lm2596_ALT
Changed lines of the file:
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@@
 			)
 		)
-		(property "Footprint" "Footprints Personalizados:Lm2596"
+		(property "Footprint" "Footprints Personalizados:Lm2596_ALT"
 			(at 105.41 55.88 0)
 			(effects

Commit message: placa semi pronta
Connections:
- net 0+: now also XT30.2 (Pin_2); no longer XT30.1 (Pin_1)
- net 5V: now also XT30_RASP1.2 (Pin_2); no longer XT30_RASP1.1 (Pin_1)
- net GND: now also XT30.1 (Pin_1), XT30_RASP1.1 (Pin_1); no longer XT30.2 (Pin_2), XT30_RASP1.2 (Pin_2)
Changed lines of the file:
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@@
 	)
 	(label "GND"
-		(at 152.4 93.98 0)
+		(at 152.4 91.44 0)
 		(effects
 			(font
@@
 			)
 			(justify left bottom)
+		)
+	)
+	(label "GND"
+		(at 39.37 74.93 180)
+		(effects
+			(font
+				(size 1.27 1.27)
+			)
+			(justify right bottom)
 		)
 	)
@@
 	)
 	(label "0+"
-		(at 39.37 74.93 180)
+		(at 39.37 72.39 180)
 		(effects
 			(font
@@
 			)
 			(justify right bottom)
-		)
-	)
-	(label "5V"
-		(at 152.4 91.44 0)
-		(effects
-			(font
-				(size 1.27 1.27)
-			)
-			(justify left bottom)
 		)
 	)
@@
 		)
 	)
-	(label "GND"
-		(at 39.37 72.39 180)
+	(label "5V"
+		(at 152.4 93.98 0)
 		(effects
 			(font
 				(size 1.27 1.27)
 			)
-			(justify right bottom)
+			(justify left bottom)
 		)
 	)

Commit message: Modificações semi finais
Parts:
- removed C_100nF1, C_100nF2: C, Capacitor_THT:C_Disc_D5.0mm_W2.5mm_P2.50mm, symbol Device:C
- removed C_470uF1, C_470uF3: C_Polarized, Capacitor_THT:CP_Radial_D10.0mm_P3.50mm, symbol Device:C_Polarized
- removed U2: XL4015, Footprints Personalizados:XL4015 DC Buck, symbol Componentes Personalizados:Lm2596
- removed XT30_RASP1: Conn_01x02_Socket, Connector_AMASS:AMASS_XT30U-M_1x02_P5.0mm_Vertical, symbol Connector:Conn_01x02_Socket

Commit message: erros ajustados e placa reformulada
Parts:
- removed C_100nF3: C, Capacitor_THT:C_Disc_D5.0mm_W2.5mm_P2.50mm, symbol Device:C
- removed C_470uF2, C_470uF4: C_Polarized, Capacitor_THT:CP_Radial_D10.0mm_P3.50mm, symbol Device:C_Polarized

Commit message: Placa Finalizada
Parts:
- added 100nf10: C, Capacitor_THT:C_Disc_D3.0mm_W1.6mm_P2.50mm, symbol Device:C
Connections:
- net BAT: now also 100nf10.1
- net GND: now also 100nf10.2
Changed lines of the file:
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@@
+		(color 0 0 0 0)
+	)
+	(junction
+		(at 26.67 87.63)
+		(diameter 0)
 		(color 0 0 0 0)
 	)
@@
 	(wire
 		(pts
-			(xy 22.86 87.63) (xy 39.37 87.63)
+			(xy 22.86 87.63) (xy 26.67 87.63)
+		)
+		(stroke
+			(width 0)
+			(type default)
+		)
+	)
+	(wire
+		(pts
+			(xy 26.67 87.63) (xy 39.37 87.63)
 		)
 		(stroke
@@
 	)
 	(symbol
+		(lib_id "Device:C")
+		(at 26.67 91.44 0)
+		(unit 1)
+		(exclude_from_sim no)
+		(in_bom yes)
+		(on_board yes)
+		(dnp no)
+		(property "Reference" "100nf10"
+			(at 33.274 93.98 0)
+			(effects
+				(font
+					(size 1.27 1.27)
+				)
+			)
+		)
+		(property "Value" "C"
+			(at 28.448 93.98 0)
+			(effects
+				(font
+					(size 1.27 1.27)
+				)
+			)
+		)
+		(property "Footprint" "Capacitor_THT:C_Disc_D3.0mm_W1.6mm_P2.50mm"
+			(at 27.6352 95.25 0)
+			(effects
+				(font
+					(size 1.27 1.27)
+				)
+				(hide yes)
+			)
+		)
+		(property "Datasheet" "~"
+			(at 26.67 91.44 0)
+			(effects
+				(font
+					(size 1.27 1.27)
+				)
+				(hide yes)
+			)
+		)
+		(property "Description" "Unpolarized capacitor"
+			(at 26.67 91.44 0)
+			(effects
+				(font
+					(size 1.27 1.27)
+				)
+				(hide yes)
+			)
+		)
+		(pin "1"
+		)
+		(pin "2"
+		)
+		(instances
+			(project "AntaresMainV6"
+				(path "/249a3426-39cb-4659-b770-3d6abd5cd250/04caba75-d4d9-4708-a614-98dfb451e114"
+					(reference "100nf10")
+					(unit 1)
+				)
+			)
+		)
+	)
+	(symbol
 		(lib_id "Componentes Personalizados:Lm2596")
 		(at 105.41 55.88 0)
@@
 					(unit 1)
 				)
+			)
+		)
+	)
+	(symbol
+		(lib_id "power:Earth")
+		(at 26.67 95.25 0)
+		(unit 1)
+		(exclude_from_sim no)
+		(in_bom yes)
+		(on_board yes)
+		(dnp no)
+		(fields_autoplaced yes)
+		(property "Reference" "#PWR013"
+			(at 26.67 101.6 0)
+			(effects
+				(font
+					(size 1.27 1.27)
+				)
+				(hide yes)
+			)
+		)
+		(property "Value" "GND"
+			(at 26.67 100.33 0)
+			(effects
+				(font
+					(size 1.27 1.27)
+				)
+			)
+		)
+		(property "Footprint" ""
+			(at 26.67 95.25 0)
+			(effects
+				(font
+					(size 1.27 1.27)
+				)
+				(hide yes)
+			)
+		)
+		(property "Datasheet" "~"
+			(at 26.67 95.25 0)
+			(effects
+				(font
+					(size 1.27 1.27)
+				)
+				(hide yes)
+			)
+		)
+		(property "Description" "Power symbol creates a global label with name \"Earth\""
+			(at 26.67 95.25 0)
+			(effects
+				(font
+					(size 1.27 1.27)
+				)
+				(hide yes)
+			)
+		)
+		(pin "1"
+		)
+		(instances
+			(project "AntaresMainV6"
+				(path "/249a3426-39cb-4659-b770-3d6abd5cd250/04caba75-d4d9-4708-a614-98dfb451e114"
+					(reference "#PWR013")
+					(unit 1)
+				)
