File: AntaresMainV6.kicad_pcb (KiCad board)
At the start: 2 copper layers, 30 parts, among them U1 Lm2596 DC-DC Buck, U2 XL4015, U3 ESP32-DEVKIT-V1, U4 DRV8833, U5 Cd74hc4067

Commit message: Mudanças nos footprints
Parts:
- added J1: Conn_01x03_Socket, Connector_JST:JST_XH_B3B-XH-A_1x03_P2.50mm_Vertical, F.Cu at (61.6, 89.0)
- added J2: Conn_01x03_Socket, Connector_JST:JST_XH_B3B-XH-A_1x03_P2.50mm_Vertical, F.Cu at (61.6, 96.8)
- TCA1: footprint Footprints Personalizados:TCA9548 -> Footprints Personalizados:TCA9548_ALT
- U1: footprint Footprints Personalizados:Lm2596 -> Footprints Personalizados:Lm2596_ALT
- moved Motor1 111.1 mm to (116.1, 25.3)
- moved Motor2 111.1 mm to (116.1, 33.1)
- moved 470uF1 94.6 mm to (62.4, 129.3)
- moved HC-SR04 94.6 mm to (61.6, 119.1)
- moved RaspberryAL1 94.6 mm to (61.7, 104.8)
- moved RaspberryTXRX1 94.6 mm to (61.7, 112.1)
- moved 470uF2 94.4 mm to (117.0, 43.3)
- moved U4 90.3 mm to (103.9, 30.2)
- moved U3 87.8 mm to (43.1, 111.9)
- moved 2.2kohm1 78.7 mm to (71.5, 129.6)
- moved 1kohm1 78.7 mm to (71.5, 125.5)
- moved U5 54.9 mm to (102.8, 95.6)
- moved QTR-8A1 52.2 mm to (106.0, 109.6)
- moved TCS34725_1 52.2 mm to (106.0, 125.2)
- moved TCA1 52.2 mm to (92.9, 122.2)
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Connections:
- U3 pad 12: /RX -> /Echo3.3v
- U3 pad 13: /TX -> /Trig
- U3 pad 14: /SCL -> unconnected-(U3-D14-Pad14)
- U3 pad 18: unconnected-(U3-VN-Pad18) -> /IN3
- U3 pad 19: /SIG -> /IN4
- U3 pad 2: GND -> unconnected-(U3-D2-Pad2)
- U3 pad 21: /S3 -> /SDA
- U3 pad 22: /S2 -> /SCL
- U3 pad 23: /S1 -> /SV_1
- U3 pad 25: unconnected-(U3-D27-Pad25) -> /S1
- U3 pad 26: unconnected-(U3-D14-Pad26) -> /S0
- U3 pad 27: /Echo3.3v -> /SV_2
- U3 pad 4: unconnected-(U3-D2-Pad4) -> /IN1
- U3 pad 5: /IN1 -> /IN2
- U4 pad 11: (no net) -> /Motors/OUT4
- U4 pad 12: /Motors/OUT2 -> unconnected-(U4-ULT-Pad12)
- U4 pad 3: (no net) -> GND
- U4 pad 4: GND -> /0+
- U4 pad 5: /0+ -> /IN3
- U4 pad 6: (no net) -> /IN4

Commit message: placa semi pronta
Parts:
- removed 470uF1: C_Polarized, Capacitor_THT:CP_Radial_D10.0mm_P3.50mm
- removed RaspberryAL1: Conn_01x02_Socket, Connector_AMASS:AMASS_XT30U-M_1x02_P5.0mm_Vertical
- TCA1: moved to B.Cu
- moved C_470uF2 200.6 mm to (213.5, 124.2), turned to -90 degrees
- moved U3 187.5 mm to (226.5, 73.0)
- moved 2.2kohm1 181.7 mm to (244.5, 74.2), turned to -90 degrees
- moved SV_1 181.0 mm to (239.5, 122.0)
- moved 1kohm1 179.1 mm to (247.5, 92.3), turned to 90 degrees
- moved SV_2 178.7 mm to (239.5, 113.5)
- moved HC-SR04 176.0 mm to (237.0, 105.0)
- moved RaspberryTXRX1 163.4 mm to (225.0, 105.5)
- moved XT30 146.2 mm to (171.8, 142.0), turned to 180 degrees
- moved U1 141.9 mm to (185.2, 127.2)
- moved C_470uF3 112.9 mm to (124.5, 115.2)
- moved U4 112.8 mm to (191.1, 101.8), turned to 180 degrees
- moved C_470uF4 102.0 mm to (125.8, 102.1), turned to -90 degrees
- moved U5 98.9 mm to (197.5, 67.0), turned to -90 degrees
- moved XT30_RASP1 95.0 mm to (124.0, 129.5)
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- renumbered J1 to SV_1, J2 to SV_2
Connections:
- TCA1 pad SC0: /Multiplexers/SCL_S1 -> unconnected-(TCA1-SCL0-PadSC0)
- TCA1 pad SC1: /Multiplexers/SCL_S2 -> unconnected-(TCA1-SCL1-PadSC1)
- TCA1 pad SC2: /Multiplexers/SCL_IMU -> /Multiplexers/SCL_S1
- TCA1 pad SC3: (no net) -> /Multiplexers/SCL_S2
- TCA1 pad SC4: unconnected-(TCA1-SCL4-PadSC4) -> /Multiplexers/SCL_IMU
- TCA1 pad SD0: /Multiplexers/SDA_S1 -> unconnected-(TCA1-SDA0-PadSD0)
- TCA1 pad SD1: /Multiplexers/SDA_S2 -> unconnected-(TCA1-SDA1-PadSD1)
- TCA1 pad SD2: /Multiplexers/SDA_IMU -> /Multiplexers/SDA_S1
- TCA1 pad SD3: unconnected-(TCA1-SDA3-PadSD3) -> /Multiplexers/SDA_S2
- TCA1 pad SD4: unconnected-(TCA1-SDA4-PadSD4) -> /Multiplexers/SDA_IMU
- U3 pad 25: /S1 -> /S2
- U3 pad 26: /S0 -> /S3
- U3 pad 32: /S3 -> /S0
- U3 pad 33: /S2 -> /S1
- XT30 pad 1: /0+ -> GND
- XT30 pad 2: GND -> /0+
- XT30_RASP1 pad 1: /5V -> GND
- XT30_RASP1 pad 2: GND -> /5V
Routing:
- net /3.3v: track 0.00 -> 201.1 mm
- net /5V_LM: track 0.00 -> 114.2 mm
- net /SCL: track 0.00 -> 103.9 mm, vias 0 -> 3
- net /0+: track 0.00 -> 77.8 mm
- net /SDA: track 0.00 -> 67.3 mm, vias 0 -> 2
- net /SIG: track 0.00 -> 64.7 mm, vias 0 -> 2
- net /IN4: track 0.00 -> 59.7 mm, vias 0 -> 2
- net /IN3: track 0.00 -> 58.2 mm, vias 0 -> 2
- net /SV_2: track 0.00 -> 54.1 mm
- net /Trig: track 0.00 -> 52.4 mm
- net /S0: track 0.00 -> 52.3 mm
- net /S1: track 0.00 -> 50.3 mm
- net /IN1: track 0.00 -> 48.6 mm
- net /S2: track 0.00 -> 48.4 mm
- net /SV_1: track 0.00 -> 46.6 mm, vias 0 -> 2
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- added copper zone on B.Cu, net GND
Other:
- board outline added: 100 x 100 mm

Commit message: Modificações semi finais
Parts:
- removed C_100nF1, C_100nF2: C, Capacitor_THT:C_Disc_D5.0mm_W2.5mm_P2.50mm
- removed C_470uF1, C_470uF3: C_Polarized, Capacitor_THT:CP_Radial_D10.0mm_P3.50mm
- removed RaspberryTXRX1, XT30_RASP1: Conn_01x02_Socket, Connector_AMASS:AMASS_XT30U-M_1x02_P5.0mm_Vertical
- removed U2: XL4015, Footprints Personalizados:XL4015 DC Buck
- added Extra_1: Conn_01x04_Socket, Connector_JST:JST_XH_B4B-XH-A_1x04_P2.50mm_Vertical, F.Cu at (176.2, 84.5)
- added Extra_2: Conn_01x04_Socket, Connector_JST:JST_XH_B4B-XH-A_1x04_P2.50mm_Vertical, F.Cu at (176.2, 76.0)
- added Extra_3: Conn_01x04_Socket, Connector_JST:JST_XH_B4B-XH-A_1x04_P2.50mm_Vertical, F.Cu at (224.5, 113.5)
- added REF**: MountingHole_3.2mm_M3_ISO7380, MountingHole:MountingHole_3.2mm_M3_ISO7380, F.Cu at (157.6, 53.0)
- added REF**: MountingHole_3.2mm_M3_ISO7380, MountingHole:MountingHole_3.2mm_M3_ISO7380, F.Cu at (243.4, 53.0)
- added REF**: MountingHole_3.2mm_M3_ISO7380, MountingHole:MountingHole_3.2mm_M3_ISO7380, F.Cu at (243.4, 138.9)
- added REF**: MountingHole_3.2mm_M3_ISO7380, MountingHole:MountingHole_3.2mm_M3_ISO7380, F.Cu at (157.6, 138.9)
- added RaspCOM1: Conn_01x03_Socket, Connector_JST:JST_XH_B3B-XH-A_1x03_P2.50mm_Vertical, F.Cu at (225.5, 105.0)
- C_470uF4: moved to B.Cu
- moved 47kOhm1 183.6 mm to (233.3, 135.0), turned to 180 degrees
- moved 100kOhm1 163.5 mm to (210.2, 135.0)
- moved C_100nF3 67.7 mm to (102.5, 126.0)
- moved Motor2 28.1 mm to (202.0, 100.5)
- moved Motor1 28.0 mm to (202.0, 92.5)
- moved C_470uF4 12.6 mm to (128.0, 114.5), turned to 0 degrees
- moved 1kohm1 0.50 mm to (247.0, 92.3)
Connections:
- TCA1 pad SC5: unconnected-(TCA1-SCL5-PadSC5) -> /Multiplexers/SCL_5
- TCA1 pad SC6: unconnected-(TCA1-SCL6-PadSC6) -> /Multiplexers/SCL_6
- TCA1 pad SC7: unconnected-(TCA1-SCL7-PadSC7) -> /Multiplexers/SCL_7
- TCA1 pad SD5: unconnected-(TCA1-SDA5-PadSD5) -> /Multiplexers/SDA_5
- TCA1 pad SD6: unconnected-(TCA1-SDA6-PadSD6) -> /Multiplexers/SDA_6
- TCA1 pad SD7: unconnected-(TCA1-SDA7-PadSD7) -> /Multiplexers/SDA_7
Routing:
- net /BAT: track 0.00 -> 67.3 mm
- net /Multiplexers/SCL_7: track 0.00 -> 55.5 mm, vias 0 -> 4
- net /Multiplexers/SDA_7: track 0.00 -> 54.8 mm, vias 0 -> 4
- net /SCL: track 103.9 -> 69.0 mm
- net /0+: track 77.8 -> 105.2 mm
- net /Multiplexers/SDA_6: track 0.00 -> 25.4 mm
- net /Multiplexers/SCL_6: track 0.00 -> 23.0 mm
- net /3.3v: track 201.1 -> 218.7 mm
- net /Multiplexers/SCL_5: track 0.00 -> 16.8 mm
- net /Multiplexers/SDA_5: track 0.00 -> 16.3 mm
- net /Motors/OUT2: track 24.8 -> 11.2 mm
- net /Motors/OUT1: track 24.8 -> 11.8 mm
- net /Motors/OUT3: track 13.1 -> 19.1 mm
- net /Motors/OUT4: track 13.1 -> 18.4 mm
- net /RX: track 30.6 -> 33.4 mm
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
Commit message: Faltando apenas LED e verificação
Parts:
- renumbered U5 to CD7H, U4 to DRV8833, U3 to ESP32, U1 to LM2596
Other:
- board text added: "+"
- board text added: "-"

Commit message: Decisão final da multiplexadora
Parts:
- added LEDs1: Conn_01x03_Socket, Connector_JST:JST_XH_B3B-XH-A_1x03_P2.50mm_Vertical, F.Cu at (227.0, 122.0)
- renumbered LM2596 to U1, ESP32 to U3, DRV8833 to U4, CD7H to U5
Connections:
- U3 pad 14: unconnected-(U3-D14-Pad14) -> /LED
Routing:
- net /LED: track 0.00 -> 60.7 mm, vias 0 -> 2
- net /5V_LM: track 114.2 -> 116.5 mm

Commit message: Remoção da mux
Parts:
- removed U5: Cd74hc4067, Footprints Personalizados:CD7_TRUE
- added Extra_4: Conn_01x03_Socket, Connector_JST:JST_XH_B3B-XH-A_1x03_P2.50mm_Vertical, F.Cu at (188.0, 59.0)
- moved QTR-8A1 25.0 mm to (179.5, 60.0), turned to 180 degrees
Connections:
- QTR-8A1 pad 10: /Multiplexers/OUT8 -> /OUT8
- QTR-8A1 pad 3: /Multiplexers/OUT1 -> /OUT1
- QTR-8A1 pad 4: /Multiplexers/OUT2 -> /OUT2
- QTR-8A1 pad 5: /Multiplexers/OUT3 -> /OUT3
- QTR-8A1 pad 6: /Multiplexers/OUT4 -> /OUT4
- QTR-8A1 pad 7: /Multiplexers/OUT5 -> /OUT5
- QTR-8A1 pad 8: /Multiplexers/OUT6 -> /OUT6
- QTR-8A1 pad 9: /Multiplexers/OUT7 -> /OUT7
- U3 pad 15: unconnected-(U3-D15-Pad15) -> /OUT8
- U3 pad 2: unconnected-(U3-D2-Pad2) -> /Extra
- U3 pad 25: /S2 -> /OUT4
- U3 pad 26: /S3 -> /OUT5
- U3 pad 32: /S0 -> /OUT1
- U3 pad 33: /S1 -> /OUT2
- U3 pad 34: /SIG -> /OUT3
- U3 pad VN: unconnected-(U3-PadVN) -> /OUT7
- U3 pad VP: unconnected-(U3-PadVP) -> /OUT6
Routing:
- net /OUT7: track 0.00 -> 103.9 mm, vias 0 -> 1
- net /OUT6: track 0.00 -> 103.1 mm, vias 0 -> 1
- net /OUT5: track 0.00 -> 95.0 mm, vias 0 -> 1
- net /OUT3: track 0.00 -> 93.8 mm, vias 0 -> 1
- net /OUT4: track 0.00 -> 91.4 mm, vias 0 -> 1
- net /OUT2: track 0.00 -> 86.5 mm, vias 0 -> 1
- net /OUT1: track 0.00 -> 85.5 mm, vias 0 -> 1
- net /OUT8: track 0.00 -> 69.5 mm
- net /SIG: track 64.7 -> 0.00 mm, vias 2 -> 0
- net /S0: track 52.3 -> 0.00 mm
- net /S1: track 50.3 -> 0.00 mm
- net /S2: track 48.4 -> 0.00 mm
- net /S3: track 46.5 -> 0.00 mm
- net /Multiplexers/OUT1: track 33.6 -> 0.00 mm
- net /Multiplexers/OUT2: track 31.3 -> 0.00 mm
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
Commit message: erros ajustados e placa reformulada
Parts:
- removed C_100nF3: C, Capacitor_THT:C_Disc_D5.0mm_W2.5mm_P2.50mm
- removed C_470uF2, C_470uF4: C_Polarized, Capacitor_THT:CP_Radial_D10.0mm_P3.50mm
- removed Extra_4: Conn_01x03_Socket, Connector_JST:JST_XH_B3B-XH-A_1x03_P2.50mm_Vertical
- removed XT30: Conn_01x02_Socket, Connector_AMASS:AMASS_XT30U-M_1x02_P5.0mm_Vertical
- added + 7.4V XT30: Conn_01x02_Socket, Connector_AMASS:AMASS_XT30U-M_1x02_P5.0mm_Vertical, F.Cu at (173.5, 140.5)
- added SV_3: Conn_01x03_Socket, Connector_JST:JST_XH_B3B-XH-A_1x03_P2.50mm_Vertical, F.Cu at (238.5, 130.5)
- moved 470uF2 61.7 mm to (215.0, 109.5), turned to 180 degrees
- moved Extra_3 60.0 mm to (189.2, 65.0)
- moved Motor2 42.0 mm to (230.2, 131.5), turned to 180 degrees
- moved Motor1 41.6 mm to (230.2, 123.0), turned to 180 degrees
- moved DRV8833 31.1 mm to (213.1, 123.8), turned to 0 degrees
- moved LEDs1 20.5 mm to (238.5, 105.0)
- moved TCA1 16.1 mm to (183.0, 98.5)
- moved QTR-8A1 15.9 mm to (164.0, 56.5), turned to 0 degrees
- moved Extra_1 13.2 mm to (189.2, 82.0)
- moved Extra_2 13.2 mm to (189.2, 73.5)
- moved MPU6050 9.82 mm to (164.0, 65.0)
- moved TCS34725_1 9.82 mm to (164.0, 82.0)
- moved TCS34725_2 9.82 mm to (164.0, 73.5)
- moved HC-SR04 9.10 mm to (238.5, 96.0)
- moved LM2596 8.84 mm to (177.5, 123.0)
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- renumbered U4 to DRV8833, U1 to LM2596
Connections:
- Extra_3 pad 1: /Multiplexers/SDA_7 -> GND
- Extra_3 pad 2: /Multiplexers/SCL_7 -> /3.3v
- Extra_3 pad 3: /3.3v -> /Multiplexers/SDA_7
- Extra_3 pad 4: GND -> /Multiplexers/SCL_7
- RaspCOM1 pad 2: /RX -> /TX
- RaspCOM1 pad 3: /TX -> /RX
- U3 pad 18: /IN3 -> /IN4
- U3 pad 19: /IN4 -> /IN3
- U3 pad 2: /Extra -> /SV_3
- U3 pad 21: /SDA -> /SCL
- U3 pad 22: /SCL -> /SDA
- U3 pad 25: /OUT4 -> /OUT2
- U3 pad 26: /OUT5 -> /OUT1
- U3 pad 32: /OUT1 -> /OUT4
- U3 pad 33: /OUT2 -> /OUT3
- U3 pad 34: /OUT3 -> /OUT5
- U3 pad VN: /OUT7 -> /OUT6
- U3 pad VP: /OUT6 -> /OUT7
Routing:
- net /SV_3: track 0.00 -> 113.4 mm, vias 0 -> 1
- net /SV_1: track 46.6 -> 117.9 mm
- net /SDA: track 69.2 -> 23.9 mm, vias 2 -> 0
- net /OUT8: track 69.5 -> 29.8 mm
- net /SCL: track 69.0 -> 31.9 mm, vias 3 -> 0
- net /OUT7: track 103.9 -> 70.7 mm, vias 1 -> 0
- net /OUT6: track 103.1 -> 71.9 mm, vias 1 -> 0
- net /Multiplexers/SCL_7: track 55.5 -> 28.6 mm, vias 4 -> 0
- net /Multiplexers/SDA_7: track 54.8 -> 30.1 mm, vias 4 -> 0
- net /Extra: track 23.3 -> 0.00 mm, vias 1 -> 0
- net /OUT5: track 95.0 -> 72.9 mm, vias 1 -> 0
- net /IN3: track 60.1 -> 39.9 mm, vias 2 -> 0
- net /OUT3: track 93.8 -> 73.9 mm, vias 1 -> 0
- net /OUT4: track 91.4 -> 72.8 mm, vias 1 -> 0
- net /IN4: track 61.6 -> 43.5 mm, vias 2 -> 0
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
Commit message: Placa Finalizada
Parts:
- added 100nf1: C, Capacitor_THT:C_Disc_D3.0mm_W1.6mm_P2.50mm, B.Cu at (164.0, 69.8)
- added 100nf10: C, Capacitor_THT:C_Disc_D3.0mm_W1.6mm_P2.50mm, B.Cu at (234.8, 84.5)
- added 100nf2: C, Capacitor_THT:C_Disc_D3.0mm_W1.6mm_P2.50mm, F.Cu at (197.5, 109.8)
- added 100nf3: C, Capacitor_THT:C_Disc_D3.0mm_W1.6mm_P2.50mm, B.Cu at (191.8, 69.8)
- added 100nf4: C, Capacitor_THT:C_Disc_D3.0mm_W1.6mm_P2.50mm, B.Cu at (191.8, 78.2)
- added 100nf6: C, Capacitor_THT:C_Disc_D3.0mm_W1.6mm_P2.50mm, B.Cu at (171.8, 78.4)
- added 100nf7: C, Capacitor_THT:C_Disc_D3.0mm_W1.6mm_P2.50mm, B.Cu at (169.0, 69.8)
- added 100nf8: C, Capacitor_THT:C_Disc_D3.0mm_W1.6mm_P2.50mm, B.Cu at (194.0, 59.0)
- added 100nf9: C, Capacitor_THT:C_Disc_D3.0mm_W1.6mm_P2.50mm, B.Cu at (235.0, 64.6)
- added Astro: LOGO, Footprints Personalizados:PCBIcon, F.Cu at (151.3, 99.5)
- XT30: renamed from + 7.4V XT30
- renumbered LM2596 to U1, DRV8833 to U4
Routing:
- net /3.3v: track 219.3 -> 221.7 mm
- net /BAT: track 74.6 -> 76.5 mm
Other:
- board text added: "Antares-Core 2026"
- board text added: "RX"
- board text added: "TX"
