File: AntaresMainV6.kicad_sch (KiCad schematic)
At the start: 7 parts, among them U3 ESP32-DEVKIT-V1

Commit message: Mudanças nos footprints
Parts:
- added J1, J2: Conn_01x03_Socket, Connector_JST:JST_XH_B3B-XH-A_1x03_P2.50mm_Vertical, symbol Connector:Conn_01x03_Socket
- U3: footprint ESP32-DEVKIT-V1:MODULE_ESP32_DEVKIT_V1 -> Footprints Personalizados:MODULE_ESP32_DEVKIT_V1
Connections:
- net 5V_LM: now also J1.2 (Pin_2), J2.2 (Pin_2)
- net GND: now also J1.1 (Pin_1), J2.1 (Pin_1)
- net SV_1: now reaches U3.23 (D23)
- net SV_1: now also J1.3 (Pin_3)
- net SV_2: now reaches U3.27 (D27)
- net SV_2: now also J2.3 (Pin_3)

Commit message: placa semi pronta
Parts:
- removed 470uF1: C_Polarized, Capacitor_THT:CP_Radial_D10.0mm_P3.50mm, symbol Device:C_Polarized
- removed RaspberryAL1: Conn_01x02_Socket, Connector_AMASS:AMASS_XT30U-M_1x02_P5.0mm_Vertical, symbol Connector:Conn_01x02_Socket
- renumbered J1 to SV_1, J2 to SV_2
Connections:
- net S0: now also U3.32 (D32); no longer U3.26 (D26)
- net S1: now also U3.33 (D33); no longer U3.25 (D25)
- net S2: now also U3.25 (D25); no longer U3.33 (D33)
- net S3: now also U3.26 (D26); no longer U3.32 (D32)

Commit message: Modificações semi finais
Parts:
- removed RaspberryTXRX1: Conn_01x02_Socket, Connector_AMASS:AMASS_XT30U-M_1x02_P5.0mm_Vertical, symbol Connector:Conn_01x02_Socket
- added RaspCOM1: Conn_01x03_Socket, Connector_JST:JST_XH_B3B-XH-A_1x03_P2.50mm_Vertical, symbol Connector:Conn_01x03_Socket
Connections:
- net GND: now also RaspCOM1.1 (Pin_1)
- net RX: now also RaspCOM1.2 (Pin_2)
- net TX: now also RaspCOM1.3 (Pin_3)
Other:
- sheet Alimentação ports: added none; removed 5V
Changed lines of the file:
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@@
-	)
-	(bus_entry
-		(at 97.79 26.67)
-		(size -2.54 2.54)
-		(stroke
-			(width 0)
-			(type default)
-		)
 	)
 	(bus_entry
@@
 	)
 	(bus_entry
+		(at 148.59 96.52)
+		(size 2.54 2.54)
+		(stroke
+			(width 0)
+			(type default)
+		)
+	)
+	(bus_entry
 		(at 97.79 83.82)
 		(size -2.54 2.54)
@@
 	(bus
 		(pts
+			(xy 148.59 96.52) (xy 148.59 99.06)
+		)
+		(stroke
+			(width 0)
+			(type default)
+		)
+	)
+	(bus
+		(pts
 			(xy 97.79 86.36) (xy 97.79 91.44)
 		)
@@
 	(bus
 		(pts
-			(xy 97.79 25.4) (xy 97.79 26.67)
+			(xy 97.79 25.4) (xy 97.79 30.48)
 		)
 		(stroke
@@
 		)
 	)
-	(wire
-		(pts
-			(xy 87.63 29.21) (xy 95.25 29.21)
-		)
-		(stroke
-			(width 0)
-			(type default)
-		)
-	)
 	(bus
 		(pts
@@
 	(bus
 		(pts
-			(xy 148.59 91.44) (xy 148.59 99.06)
+			(xy 148.59 91.44) (xy 148.59 96.52)
 		)
 		(stroke
@@
 	(wire
 		(pts
+			(xy 151.13 99.06) (xy 166.37 99.06)
+		)
+		(stroke
+			(width 0)
+			(type default)
+		)
+	)
+	(wire
+		(pts
 			(xy 100.33 27.94) (xy 106.68 27.94)
 		)
@@
 		(pts
 			(xy 87.63 96.52) (xy 95.25 96.52)
-		)
-		(stroke
-			(width 0)
-			(type default)
-		)
-	)
-	(bus
-		(pts
-			(xy 97.79 26.67) (xy 97.79 30.48)
 		)
 		(stroke
@@
 		)
 	)
-	(label "5V"
-		(at 95.25 29.21 180)
-		(effects
-			(font
-				(size 1.27 1.27)
-			)
-			(justify right bottom)
-		)
-	)
 	(label "IN4"
 		(at 100.33 127 0)
@@
 			)
 			(justify right bottom)
+		)
+	)
+	(label "GND"
+		(at 151.13 99.06 0)
+		(effects
+			(font
+				(size 1.27 1.27)
+			)
+			(justify left bottom)
 		)
 	)
@@
 	)
 	(symbol
+		(lib_id "Connector:Conn_01x03_Socket")
+		(at 171.45 101.6 0)
+		(unit 1)
+		(exclude_from_sim no)
+		(in_bom yes)
+		(on_board yes)
+		(dnp no)
+		(fields_autoplaced yes)
+		(property "Reference" "RaspCOM1"
+			(at 172.72 100.3299 0)
+			(effects
+				(font
+					(size 1.27 1.27)
+				)
+				(justify left)
+			)
+		)
+		(property "Value" "Conn_01x03_Socket"
+			(at 172.72 102.8699 0)
+			(effects
+				(font
+					(size 1.27 1.27)
+				)
+				(justify left)
+			)
+		)
+		(property "Footprint" "Connector_JST:JST_XH_B3B-XH-A_1x03_P2.50mm_Vertical"
+			(at 171.45 101.6 0)
+			(effects
+				(font
+					(size 1.27 1.27)
+				)
+				(hide yes)
+			)
+		)
+		(property "Datasheet" "~"
+			(at 171.45 101.6 0)
+			(effects
+				(font
+					(size 1.27 1.27)
+				)
+				(hide yes)
+			)
+		)
+		(property "Description" "Generic connector, single row, 01x03, script generated"
+			(at 171.45 101.6 0)
+			(effects
+				(font
+					(size 1.27 1.27)
+				)
+				(hide yes)
+			)
+		)
+		(pin "2"
+		)
+		(pin "3"
+		)
+		(pin "1"
+		)
+		(instances
+			(project "AntaresMainV6"
+				(path "/249a3426-39cb-4659-b770-3d6abd5cd250"
+					(reference "RaspCOM1")
+					(unit 1)
+				)
+			)
+		)
+	)
+	(symbol
 		(lib_id "Device:R")
 		(at 87.63 125.73 180)
@@
 	)
 	(symbol
-		(lib_id "Connector:Conn_01x02_Socket")
-		(at 171.45 101.6 0)
-		(unit 1)
-		(exclude_from_sim no)
-		(in_bom yes)
-		(on_board yes)
-		(dnp no)
-		(fields_autoplaced yes)
-		(property "Reference" "RaspberryTXRX1"
-			(at 172.72 101.5999 0)
-			(effects
-				(font
-					(size 1.27 1.27)
-				)
-				(justify left)
-			)
-		)
-		(property "Value" "Conn_01x02_Socket"
-			(at 172.72 104.1399 0)
-			(effects
-				(font
-					(size 1.27 1.27)
-				)
-				(justify left)
-			)
-		)
-		(property "Footprint" "Connector_AMASS:AMASS_XT30U-M_1x02_P5.0mm_Vertical"
-			(at 171.45 101.6 0)
-			(effects
-				(font
-					(size 1.27 1.27)
-				)
-				(hide yes)
-			)
-		)
-		(property "Datasheet" "~"
-			(at 171.45 101.6 0)
-			(effects
-				(font
-					(size 1.27 1.27)
-				)
-				(hide yes)
-			)
-		)
-		(property "Description" "Generic connector, single row, 01x02, script generated"
-			(at 171.45 101.6 0)
-			(effects
-				(font
-					(size 1.27 1.27)
-				)
-				(hide yes)
-			)
-		)
-		(pin "1"
-		)
-		(pin "2"
-		)
-		(instances
-			(project ""
-				(path "/249a3426-39cb-4659-b770-3d6abd5cd250"
-					(reference "RaspberryTXRX1")
-					(unit 1)
-				)
-			)
-		)
-	)
-	(symbol
 		(lib_id "power:Earth")
 		(at 68.58 134.62 0)
@@
 			)
 		)
-		(pin "5V" output
-			(at 87.63 29.21 0)
-			(effects
-				(font
-					(size 1.27 1.27)
-				)
-				(justify right)
-			)
-		)

Commit message: Decisão final da multiplexadora
Parts:
- added LEDs1: Conn_01x03_Socket, Connector_JST:JST_XH_B3B-XH-A_1x03_P2.50mm_Vertical, symbol Connector:Conn_01x03_Socket
Connections:
- net 5V_LM: now also LEDs1.2 (Pin_2)
- net GND: now also LEDs1.1 (Pin_1)
- net LED: now reaches U3.14 (D14)
- net LED: now also LEDs1.3 (Pin_3)
Changed lines of the file:
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@@
+	)
+	(bus_entry
+		(at 97.79 116.84)
+		(size 2.54 2.54)
+		(stroke
+			(width 0)
+			(type default)
+		)
 	)
 	(bus_entry
@@
 	)
 	(bus_entry
+		(at 148.59 130.81)
+		(size 2.54 2.54)
+		(stroke
+			(width 0)
+			(type default)
+		)
+	)
+	(bus_entry
 		(at 97.79 40.64)
 		(size 2.54 2.54)
@@
 	)
 	(bus_entry
+		(at 148.59 128.27)
+		(size 2.54 2.54)
+		(stroke
+			(width 0)
+			(type default)
+		)
+	)
+	(bus_entry
 		(at 148.59 116.84)
 		(size -2.54 2.54)
@@
 	)
 	(bus_entry
+		(at 148.59 125.73)
+		(size 2.54 2.54)
+		(stroke
+			(width 0)
+			(type default)
+		)
+	)
+	(bus_entry
 		(at 148.59 88.9)
 		(size -2.54 2.54)
@@
 	(bus
 		(pts
-			(xy 148.59 124.46) (xy 148.59 132.08)
+			(xy 148.59 124.46) (xy 148.59 125.73)
 		)
 		(stroke
@@
 	(bus
 		(pts
+			(xy 97.79 116.84) (xy 97.79 121.92)
+		)
+		(stroke
+			(width 0)
+			(type default)
+		)
+	)
+	(bus
+		(pts
 			(xy 148.59 109.22) (xy 148.59 110.49)
 		)
@@
 		)
 	)
+	(wire
+		(pts
+			(xy 151.13 128.27) (xy 166.37 128.27)
+		)
+		(stroke
+			(width 0)
+			(type default)
+		)
+	)
 	(bus
 		(pts
@@
 	(bus
 		(pts
+			(xy 148.59 125.73) (xy 148.59 128.27)
+		)
+		(stroke
+			(width 0)
+			(type default)
+		)
+	)
+	(bus
+		(pts
 			(xy 148.59 104.14) (xy 148.59 105.41)
 		)
@@
 	(wire
 		(pts
+			(xy 151.13 130.81) (xy 166.37 130.81)
+		)
+		(stroke
+			(width 0)
+			(type default)
+		)
+	)
+	(wire
+		(pts
 			(xy 87.63 118.11) (xy 95.25 118.11)
 		)
@@
 	(wire
 		(pts
+			(xy 151.13 133.35) (xy 166.37 133.35)
+		)
+		(stroke
+			(width 0)
+			(type default)
+		)
+	)
+	(wire
+		(pts
 			(xy 151.13 101.6) (xy 166.37 101.6)
 		)
@@
 	(wire
 		(pts
+			(xy 100.33 119.38) (xy 111.76 119.38)
+		)
+		(stroke
+			(width 0)
+			(type default)
+		)
+	)
+	(wire
+		(pts
 			(xy 142.24 93.98) (xy 146.05 93.98)
 		)
@@
 	(bus
 		(pts
+			(xy 148.59 128.27) (xy 148.59 130.81)
+		)
+		(stroke
+			(width 0)
+			(type default)
+		)
+	)
+	(bus
+		(pts
 			(xy 148.59 118.11) (xy 148.59 119.38)
 		)
@@
 	(bus
 		(pts
+			(xy 148.59 130.81) (xy 148.59 132.08)
+		)
+		(stroke
+			(width 0)
+			(type default)
+		)
+	)
+	(bus
+		(pts
 			(xy 97.79 106.68) (xy 97.79 109.22)
 		)
@@
 	(bus
 		(pts
-			(xy 97.79 115.57) (xy 97.79 121.92)
+			(xy 97.79 115.57) (xy 97.79 116.84)
 		)
 		(stroke
@@
 		)
 	)
+	(label "LED"
+		(at 151.13 133.35 0)
+		(effects
+			(font
+				(size 1.27 1.27)
+			)
+			(justify left bottom)
+		)
+	)
 	(label "IN4"
 		(at 95.25 86.36 180)
@@
 		)
 	)
+	(label "GND"
+		(at 151.13 128.27 0)
+		(effects
+			(font
+				(size 1.27 1.27)
+			)
+			(justify left bottom)
+		)
+	)
 	(label "SV_1"
 		(at 146.05 109.22 180)
@@
 		)
 	)
+	(label "LED"
+		(at 100.33 119.38 0)
+		(effects
+			(font
+				(size 1.27 1.27)
+			)
+			(justify left bottom)
+		)
+	)
 	(label "IN2"
 		(at 95.25 93.98 180)
@@
 			)
 			(justify right bottom)
+		)
+	)
+	(label "5V_LM"
+		(at 151.13 130.81 0)
+		(effects
+			(font
+				(size 1.27 1.27)
+			)
+			(justify left bottom)
 		)
 	)
@@
 					(unit 1)
 				)
+			)
+		)
+	)
+	(symbol
+		(lib_id "Connector:Conn_01x03_Socket")
+		(at 171.45 130.81 0)
+		(unit 1)
+		(exclude_from_sim no)
+		(in_bom yes)
+		(on_board yes)
+		(dnp no)
+		(fields_autoplaced yes)
+		(property "Reference" "LEDs1"
+			(at 172.72 129.5399 0)
+			(effects
+				(font
+					(size 1.27 1.27)
+				)
+				(justify left)
+			)
+		)
+		(property "Value" "Conn_01x03_Socket"
+			(at 172.72 132.0799 0)
+			(effects
+				(font
+					(size 1.27 1.27)
+				)
+				(justify left)
+			)
+		)
+		(property "Footprint" "Connector_JST:JST_XH_B3B-XH-A_1x03_P2.50mm_Vertical"
+			(at 171.45 130.81 0)
+			(effects
+				(font
+					(size 1.27 1.27)
+				)
+				(hide yes)
+			)
+		)
+		(property "Datasheet" "~"
+			(at 171.45 130.81 0)
+			(effects
+				(font
+					(size 1.27 1.27)
+				)
+				(hide yes)
+			)
+		)
+		(property "Description" "Generic connector, single row, 01x03, script generated"
+			(at 171.45 130.81 0)
+			(effects
+				(font
+					(size 1.27 1.27)
+				)
+				(hide yes)
+			)
+		)
+		(pin "2"
+		)
+		(pin "3"
+		)
+		(pin "1"
+		)
+		(instances
+			(project "AntaresMainV6"
+				(path "/249a3426-39cb-4659-b770-3d6abd5cd250"
+					(reference "LEDs1")
+					(unit 1)
+				)

Commit message: Remoção da mux
Parts:
- added Extra_4: Conn_01x03_Socket, Connector_JST:JST_XH_B3B-XH-A_1x03_P2.50mm_Vertical, symbol Connector:Conn_01x03_Socket
- added QTR-8A1: Conn_01x11_Socket, Connector_JST:JST_XH_B11B-XH-A_1x11_P2.50mm_Vertical, symbol Connector:Conn_01x11_Socket
Connections:
- net 3.3v: now also Extra_4.2 (Pin_2), QTR-8A1.11 (Pin_11), QTR-8A1.2 (Pin_2)
- net GND: now also Extra_4.1 (Pin_1), QTR-8A1.1 (Pin_1)
- net S0: no longer U3.32 (D32)
- net S1: no longer U3.33 (D33)
- net S2: no longer U3.25 (D25)
- net S3: no longer U3.26 (D26)
- net SIG: no longer U3.34 (D34)
- net OUT8: now reaches U3.15 (D15)
- net OUT8: now also QTR-8A1.10 (Pin_10)
- net Extra: now reaches U3.2 (D2)
- net Extra: now also Extra_4.3 (Pin_3)
- net OUT7: now reaches U3.VN
- net OUT7: now also QTR-8A1.9 (Pin_9)
- net OUT6: now reaches U3.VP
- net OUT6: now also QTR-8A1.8 (Pin_8)
- new net OUT1: QTR-8A1.3 (Pin_3), U3.32 (D32)
- new net OUT2: QTR-8A1.4 (Pin_4), U3.33 (D33)
- new net OUT3: QTR-8A1.5 (Pin_5), U3.34 (D34)
- new net OUT4: QTR-8A1.6 (Pin_6), U3.25 (D25)
- new net OUT5: QTR-8A1.7 (Pin_7), U3.26 (D26)
- no-connect marks 5 -> 3

Commit message: erros ajustados e placa reformulada
Parts:
- renumbered Extra_4 to SV_3
Connections:
- net 3.3v: no longer SV_3.2 (Pin_2)
- net 5V_LM: now also SV_3.2 (Pin_2)
- net IN3: now also U3.19 (D19); no longer U3.18 (D18)
- net IN4: now also U3.18 (D18); no longer U3.19 (D19)
- net OUT1: now also U3.26 (D26); no longer U3.32 (D32)
- net OUT2: now also U3.25 (D25); no longer U3.33 (D33)
- net OUT3: now also U3.33 (D33); no longer U3.34 (D34)
- net OUT4: now also U3.32 (D32); no longer U3.25 (D25)
- net OUT5: now also U3.34 (D34); no longer U3.26 (D26)
- net OUT6: now also U3.VN; no longer U3.VP
- net OUT7: now also U3.VP; no longer U3.VN
- net RX: now also RaspCOM1.3 (Pin_3); no longer RaspCOM1.2 (Pin_2)
- net SCL: now also U3.21 (D21); no longer U3.22 (D22)
- net SDA: now also U3.22 (D22); no longer U3.21 (D21)
- net TX: now also RaspCOM1.2 (Pin_2); no longer RaspCOM1.3 (Pin_3)
- net Extra renamed SV_3
Changed lines of the file:
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@@
 		)
 	)
-	(label "OUT3"
+	(label "OUT5"
 		(at 146.05 127 180)
 		(effects
@@
 		)
 	)
-	(label "OUT7"
+	(label "OUT6"
 		(at 100.33 95.25 0)
 		(effects
@@
 		)
 	)
-	(label "OUT5"
+	(label "OUT1"
 		(at 146.05 114.3 180)
 		(effects
@@
 		)
 	)
-	(label "Extra"
+	(label "SV_3"
 		(at 151.13 143.51 0)
 		(effects
@@
 		)
 	)
-	(label "Extra"
-		(at 101.6 106.68 0)
-		(effects
-			(font
-				(size 1.27 1.27)
-			)
-			(justify left bottom)
-		)
-	)
-	(label "RX"
+	(label "SV_3"
+		(at 100.33 106.68 0)
+		(effects
+			(font
+				(size 1.27 1.27)
+			)
+			(justify left bottom)
+		)
+	)
+	(label "TX"
 		(at 151.13 101.6 0)
 		(effects
@@
 		)
 	)
-	(label "OUT2"
+	(label "OUT3"
 		(at 146.05 121.92 180)
 		(effects
@@
 		)
 	)
-	(label "OUT6"
+	(label "OUT7"
 		(at 100.33 91.44 0)
 		(effects
@@
 		)
 	)
-	(label "SCL"
+	(label "SDA"
 		(at 146.05 106.68 180)
 		(effects
@@
 		)
 	)
-	(label "IN4"
+	(label "IN3"
 		(at 100.33 127 0)
 		(effects
@@
 		)
 	)
-	(label "3.3v"
+	(label "5V_LM"
 		(at 151.13 140.97 0)
 		(effects
@@
 		)
 	)
-	(label "SDA"
+	(label "SCL"
 		(at 100.33 129.54 0)
 		(effects
@@
 		)
 	)
-	(label "IN3"
+	(label "IN4"
 		(at 100.33 124.46 0)
 		(effects
@@
 		)
 	)
-	(label "OUT1"
+	(label "OUT4"
 		(at 146.05 119.38 180)
 		(effects
@@
 		)
 	)
-	(label "TX"
+	(label "RX"
 		(at 151.13 104.14 0)
 		(effects
@@
 		)
 	)
-	(label "OUT4"
+	(label "OUT2"
 		(at 146.05 111.76 180)
 		(effects
@@
 		(dnp no)
 		(fields_autoplaced yes)
-		(property "Reference" "Extra_4"
+		(property "Reference" "SV_3"
 			(at 172.72 139.6999 0)
 			(effects
@@
 			(project "AntaresMainV6"
 				(path "/249a3426-39cb-4659-b770-3d6abd5cd250"
-					(reference "Extra_4")
+					(reference "SV_3")
 					(unit 1)
 				)

Commit message: Placa Finalizada
Parts:
- added 100nf8, 100nf9: C, Capacitor_THT:C_Disc_D3.0mm_W1.6mm_P2.50mm, symbol Device:C
Connections:
- net 3.3v: now also 100nf8.1
- net 5V_LM: now also 100nf9.2
- net GND: now also 100nf8.2, 100nf9.1
