File: Motors.kicad_sch (KiCad schematic)
At the start: 4 parts, among them U4 DRV8833

Commit message: Mudanças nos footprints
Connections:
- net 0+: now also U4.4 (VCC); no longer U4.5 (VCC)
- net 3.3v: now also U4.7 (EEP); no longer U4.9 (EEP)
- net GND: now also U4.3 (GND); no longer U4.4 (GND)
- net IN3: now also U4.5 (IN3); no longer U4.7 (IN3)
- net IN4: now also U4.6 (IN4); no longer U4.8 (IN4)
- net OUT1: now also U4.8 (OUT1); no longer U4.10 (OUT1)
- net OUT2: now also U4.9 (OUT2); no longer U4.12 (OUT2)
- net OUT3: now also U4.10 (OUT3); no longer U4.13 (OUT3)
- net OUT4: now also U4.11 (OUT4); no longer U4.15 (OUT4)
Changed lines of the file:
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@@
 		(pin "8"
 		)
-		(pin "16"
+		(pin "6"
 		)
 		(pin "9"
@@
 		(pin "4"
 		)
-		(pin "13"
+		(pin "3"
 		)
 		(pin "10"
@@
 		(pin "12"
 		)
-		(pin "15"
+		(pin "11"
 		)
 		(pin "5"

Commit message: Placa Finalizada
Changed lines of the file:
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@@
 	(wire
 		(pts
-			(xy 153.67 85.09) (xy 137.16 85.09)
+			(xy 137.16 85.09) (xy 153.67 85.09)
 		)
 		(stroke
